Commit message: The UPdated ONEs

File: urdf/pick_place_robot.urdf.xacro (robot description, xacro)
@@ -188,14 +188,39 @@
     <limit lower="0" upper="0.04" effort="10" velocity="0.1"/>
   </joint>
-  <!-- Gazebo plugins -->
+  <!-- ros2_control -->
+  <ros2_control name="pick_place_robot_system" type="system">
+    <hardware>
+      <plugin>gazebo_ros2_control/GazeboSystem</plugin>
+    </hardware>
+    <joint name="joint1">
+      <command_interface name="position"/>
+      <state_interface name="position"/>
+      <state_interface name="velocity"/>
+    </joint>
+    <joint name="joint2">
+      <command_interface name="position"/>
+      <state_interface name="position"/>
+      <state_interface name="velocity"/>
+    </joint>
+    <joint name="joint3">
+      <command_interface name="position"/>
+      <state_interface name="position"/>
+      <state_interface name="velocity"/>
+    </joint>
+    <joint name="gripper_left_joint">
+      <command_interface name="position"/>
+      <state_interface name="position"/>
+      <state_interface name="velocity"/>
+    </joint>
+    <joint name="gripper_right_joint">
+      <command_interface name="position"/>
+      <state_interface name="position"/>
+      <state_interface name="velocity"/>
+    </joint>
+  </ros2_control>
+  <!-- Gazebo ros2_control plugin -->
   <gazebo>
-    <plugin name="gazebo_ros_control" filename="libgazebo_ros_control.so">
-      <robotNamespace>/pick_place_robot</robotNamespace>
-    </plugin>
-  </gazebo>
-  <!-- Joint state publisher -->
-  <gazebo>
-    <plugin name="joint_state_publisher" filename="libgazebo_ros_joint_state_publisher.so">
-      <jointName>joint1, joint2, joint3, gripper_left_joint, gripper_right_joint</jointName>
+    <plugin filename="libgazebo_ros2_control.so" name="gazebo_ros2_control">
+      <parameters>$(find pick_place_robot)/config/controllers.yaml</parameters>
     </plugin>
   </gazebo>
